File: CircuitoV5/CircuitoV5.kicad_pcb (KiCad board)
At the start: 2 copper layers, 43.4 x 59.6 mm, 22 parts, among them J1 Conn_01x05, J2 Conn_01x02, J3 Conn_01x02, U1 LM324, U2 LM358

Commit message: Ultimas actualizaciones y correcciones
Connections:
- C2 pad 1: Net-(C2-Pad1) -> Net-(U2B-+)
- R10 pad 1: Net-(U2B-+) -> Net-(R10-Pad1)
- R10 pad 2: Net-(C2-Pad1) -> Net-(U2B-+)
- R7 pad 2: Net-(U2B-+) -> Net-(R10-Pad1)
- U2 pad 1: Net-(U2B-+) -> Net-(R10-Pad1)
Routing:
- net Net-(U2B-+): track 20.2 -> 33.1 mm
- net Net-(R10-Pad1): track 0.00 -> 9.46 mm
- net Net-(C2-Pad1): track 8.10 -> 0.00 mm
Changed lines of the file:
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@@
 		(tags "C Disc series Radial pin pitch 2.50mm diameter 5mm width 2.5mm Capacitor")
 		(property "Reference" "C5"
-			(at 1.25 -2.5 90)
+			(at 1.7 2.5 90)
 			(layer "F.SilkS")
 			(effects
@@
 		(tags "Potentiometer vertical Bourns 3296W")
 		(property "Reference" "RV1"
-			(at -2.54 -3.66 90)
+			(at 3.785 1.675 90)
 			(layer "F.SilkS")
 			(effects
@@
 		(tags "Through hole socket strip THT 1x02 2.54mm single row")
 		(property "Reference" "J2"
-			(at 0 -2.77 90)
+			(at -0.25 5.14 270)
 			(layer "F.SilkS")
 			(effects
@@
 			(layers "*.Cu" "*.Mask")
 			(remove_unused_layers no)
-			(net "Net-(U2B-+)")
+			(net "Net-(R10-Pad1)")
 			(pintype "passive")
 		)
@@
 			(layers "*.Cu" "*.Mask")
 			(remove_unused_layers no)
-			(net "Net-(C2-Pad1)")
+			(net "Net-(U2B-+)")
 			(pintype "passive")
 		)
@@
 		(tags "Resistor Axial_DIN0207 series Axial Horizontal pin pitch 10.16mm 0.25W = 1/4W length 6.3mm diameter 2.5mm")
 		(property "Reference" "R3"
-			(at 5.08 -2.37 0)
+			(at 4.4 -2.2 0)
 			(layer "F.SilkS")
 			(effects
@@
 		(tags "THT DIP DIL PDIP 2.54mm 7.62mm 300mil")
 		(property "Reference" "U1"
-			(at 3.81 -2.33 90)
+			(at 3.91 17.56 90)
 			(layer "F.SilkS")
 			(effects
@@
 		(tags "Through hole socket strip THT 1x02 2.54mm single row")
 		(property "Reference" "J3"
-			(at 0 -2.77 90)
+			(at 0 5.025 90)
 			(layer "F.SilkS")
 			(effects
@@
 		(tags "C Disc series Radial pin pitch 2.50mm diameter 5mm width 2.5mm Capacitor")
 		(property "Reference" "C6"
-			(at 1.25 -2.5 90)
+			(at 5.125 0.1 90)
 			(layer "F.SilkS")
 			(effects
@@
 		(tags "C Disc series Radial pin pitch 2.50mm diameter 5mm width 2.5mm Capacitor")
 		(property "Reference" "C3"
-			(at 1.25 -2.5 90)
+			(at 3.9 -2.3 90)
 			(layer "F.SilkS")
 			(effects
@@
 		(tags "C Disc series Radial pin pitch 2.50mm diameter 5mm width 2.5mm Capacitor")
 		(property "Reference" "C4"
-			(at 1.25 -2.5 90)
+			(at 4.975 0 180)
 			(layer "F.SilkS")
 			(effects
@@
 		(tags "THT DIP DIL PDIP 2.54mm 7.62mm 300mil")
 		(property "Reference" "U2"
-			(at 3.81 -2.33 90)
+			(at -2.09 2.31 180)
 			(layer "F.SilkS")
 			(effects
@@
 			(remove_unused_layers no)
 			(roundrect_rratio 0.15625)
-			(net "Net-(U2B-+)")
+			(net "Net-(R10-Pad1)")
 			(pintype "output")
 		)
@@
 			(layers "*.Cu" "*.Mask")
 			(remove_unused_layers no)
-			(net "Net-(C2-Pad1)")
+			(net "Net-(U2B-+)")
 			(pintype "passive")
 		)
@@
 			(layers "*.Cu" "*.Mask")
 			(remove_unused_layers no)
-			(net "Net-(U2B-+)")
+			(net "Net-(R10-Pad1)")
 			(pintype "passive")
 		)
@@
 	)
 	(segment
-		(start 90.42 57.5)
-		(end 92.5 55.42)
+		(start 85.04 50.3)
+		(end 82.34 53)
 		(width 0.25)
 		(layer "F.Cu")
@@
 	)
 	(segment
-		(start 94.69 50.81)
-		(end 92.5 53)
+		(start 97.8 48.7)
+		(end 94.9 48.7)
 		(width 0.25)
 		(layer "F.Cu")
@@
 	)
 	(segment
-		(start 95.69 50.81)
-		(end 94.69 50.81)
+		(start 103.31 43.19)
+		(end 97.8 48.7)
 		(width 0.25)
 		(layer "F.Cu")
@@
 	)
 	(segment
-		(start 92.5 55.42)
-		(end 92.5 53)
+		(start 82.34 54.74)
+		(end 85 57.4)
 		(width 0.25)
 		(layer "F.Cu")
@@
 	)
 	(segment
-		(start 103.31 43.19)
-		(end 95.69 50.81)
+		(start 94.9 48.7)
+		(end 93.3 50.3)
 		(width 0.25)
 		(layer "F.Cu")
@@
 	)
 	(segment
-		(start 82.34 54.74)
-		(end 85 57.4)
+		(start 85 57.4)
+		(end 85 60)
 		(width 0.25)
 		(layer "F.Cu")
-		(net "Net-(C2-Pad1)")
+		(net "Net-(U2B-+)")
 	)
 	(segment
-		(start 85 57.4)
-		(end 85 60)
+		(start 93.3 50.3)
+		(end 85.04 50.3)
 		(width 0.25)
 		(layer "F.Cu")
-		(net "Net-(C2-Pad1)")
+		(net "Net-(U2B-+)")
 	)
 	(segment
@@
 		(width 0.25)
 		(layer "F.Cu")
-		(net "Net-(C2-Pad1)")
+		(net "Net-(U2B-+)")
 	)
 	(segment
@@
 		(net "Net-(U2A-+)")
 	)
+	(segment
+		(start 94.69 50.81)
+		(end 95.69 50.81)
+		(width 0.2)
+		(layer "F.Cu")
+		(net "Net-(R10-Pad1)")
+	)
+	(segment
+		(start 90.42 57.5)
+		(end 90.42 55.08)
+		(width 0.2)
+		(layer "F.Cu")
+		(net "Net-(R10-Pad1)")
+	)
+	(segment
+		(start 92.5 53)
+		(end 94.69 50.81)
+		(width 0.2)
+		(layer "F.Cu")
+		(net "Net-(R10-Pad1)")
+	)
+	(segment
+		(start 90.42 55.08)
+		(end 92.5 53)
+		(width 0.2)
+		(layer "F.Cu")
+		(net "Net-(R10-Pad1)")
+	)
 	(zone
